Commit message: vehicle and sensor urdf model fixed

File: sensor_kit/autoware_towtruck_sensor_kit_launch/autoware_towtruck_sensor_kit_description/urdf/sensor_kit.xacro (robot description, xacro)
@@ -14,7 +14,5 @@
       <child link="${sensor_kit_base_link}"/>
     </joint>
-    <link name="${sensor_kit_base_link}">
-      <origin rpy="0 0 0" xyz="0 0 0"/>
-    </link>
+    <link name="${sensor_kit_base_link}"/>
     <!-- sensor -->
     <xacro:property name="calibration" value="${xacro.load_yaml('$(arg config_dir)/sensor_kit_calibration.yaml')}"/>

File: vehicle/autoware_towtruck_vehicle_launch/autoware_towtruck_vehicle_description/urdf/vehicle.xacro (robot description, xacro)
@@ -18,4 +18,9 @@
   </joint>
   <link name="chassis_link">
+    <inertial>
+      <origin xyz="0 0 0" rpy="0 0 0"/>
+      <mass value="500.0"/>
+      <inertia ixx="100.0" ixy="0.0" ixz="0.0" iyy="100.0" iyz="0.0" izz="100.0"/>
+    </inertial>
     <visual>
       <origin xyz="0 0 0.95" rpy="0 0 0"/>

Commit message: Updating vehicle and sensor urdf model

File: sensor_kit/autoware_towtruck_sensor_kit_launch/autoware_towtruck_sensor_kit_description/urdf/sensor_kit.xacro (robot description, xacro)
@@ -2,10 +2,5 @@
 <robot xmlns:xacro="http://ros.org/wiki/xacro">
   <xacro:macro name="sensor_kit_macro" params="parent x y z roll pitch yaw">
-    <xacro:include filename="$(find velodyne_description)/urdf/VLP-16.urdf.xacro"/>
-    <xacro:include filename="$(find vls_description)/urdf/VLS-128.urdf.xacro"/>
-    <xacro:include filename="$(find camera_description)/urdf/monocular_camera.xacro"/>
-    <xacro:include filename="$(find imu_description)/urdf/imu.xacro"/>
-    <xacro:arg name="gpu" default="false"/>
-    <xacro:arg name="config_dir" default="$(find sample_sensor_kit_description)/config"/>
+    <xacro:arg name="config_dir" default="$(find autoware_towtruck_sensor_kit_description)/config"/>
     <xacro:property name="sensor_kit_base_link" default="sensor_kit_base_link"/>
     <joint name="${sensor_kit_base_link}_joint" type="fixed">
@@ -15,18 +10,11 @@
     </joint>
     <link name="${sensor_kit_base_link}"/>
-    <!-- sensor -->
     <xacro:property name="calibration" value="${xacro.load_yaml('$(arg config_dir)/sensor_kit_calibration.yaml')}"/>
-    <!-- lidar -->
-    <!-- <xacro:VLS-128 parent="sensor_kit_base_link" name="velodyne_top" topic="/points_raw" hz="10" samples="220" gpu="$(arg gpu)">
-      <origin
-        xyz="${calibration['sensor_kit_base_link']['velodyne_top_base_link']['x']}
-             ${calibration['sensor_kit_base_link']['velodyne_top_base_link']['y']}
-             ${calibration['sensor_kit_base_link']['velodyne_top_base_link']['z']}"
-        rpy="${calibration['sensor_kit_base_link']['velodyne_top_base_link']['roll']}
-             ${calibration['sensor_kit_base_link']['velodyne_top_base_link']['pitch']}
-             ${calibration['sensor_kit_base_link']['velodyne_top_base_link']['yaw']}"
-      />
-    </xacro:VLS-128> -->
-    <xacro:VLP-16 parent="sensor_kit_base_link" name="velodyne_left" topic="/points_raw" hz="10" samples="220" gpu="$(arg gpu)">
+    <!-- Livox MID-360 LiDARs — keep legacy `velodyne_*_base_link` frame names so
+         downstream rviz/localization configs don't need edits. -->
+    <link name="velodyne_left_base_link"/>
+    <joint name="velodyne_left_base_link_joint" type="fixed">
+      <parent link="sensor_kit_base_link"/>
+      <child link="velodyne_left_base_link"/>
       <origin
         xyz="${calibration['sensor_kit_base_link']['velodyne_left_base_link']['x']}
@@ -35,8 +23,10 @@
         rpy="${calibration['sensor_kit_base_link']['velodyne_left_base_link']['roll']}
              ${calibration['sensor_kit_base_link']['velodyne_left_base_link']['pitch']}
-             ${calibration['sensor_kit_base_link']['velodyne_left_base_link']['yaw']}"
-      />
-    </xacro:VLP-16>
-    <xacro:VLP-16 parent="sensor_kit_base_link" name="velodyne_right" topic="/points_raw" hz="10" samples="220" gpu="$(arg gpu)">
+             ${calibration['sensor_kit_base_link']['velodyne_left_base_link']['yaw']}"/>
+    </joint>
+    <link name="velodyne_right_base_link"/>
+    <joint name="velodyne_right_base_link_joint" type="fixed">
+      <parent link="sensor_kit_base_link"/>
+      <child link="velodyne_right_base_link"/>
       <origin
         xyz="${calibration['sensor_kit_base_link']['velodyne_right_base_link']['x']}
@@ -45,154 +35,31 @@
         rpy="${calibration['sensor_kit_base_link']['velodyne_right_base_link']['roll']}
              ${calibration['sensor_kit_base_link']['velodyne_right_base_link']['pitch']}
-             ${calibration['sensor_kit_base_link']['velodyne_right_base_link']['yaw']}"
-      />
-    </xacro:VLP-16>
-    <!-- camera -->
-    <!-- <xacro:monocular_camera_macro
-      name="traffic_light_right_camera/camera"
-      parent="sensor_kit_base_link"
-      namespace=""
-      x="${calibration['sensor_kit_base_link']['traffic_light_right_camera/camera_link']['x']}"
-      y="${calibration['sensor_kit_base_link']['traffic_light_right_camera/camera_link']['y']}"
-      z="${calibration['sensor_kit_base_link']['traffic_light_right_camera/camera_link']['z']}"
-      roll="${calibration['sensor_kit_base_link']['traffic_light_right_camera/camera_link']['roll']}"
-      pitch="${calibration['sensor_kit_base_link']['traffic_light_right_camera/camera_link']['pitch']}"
-      yaw="${calibration['sensor_kit_base_link']['traffic_light_right_camera/camera_link']['yaw']}"
-      fps="30"
-      width="800"
-      height="400"
-      fov="1.3"
-    />
-    <xacro:monocular_camera_macro
-      name="traffic_light_left_camera/camera"
-      parent="sensor_kit_base_link"
-      namespace=""
-      x="${calibration['sensor_kit_base_link']['traffic_light_left_camera/camera_link']['x']}"
-      y="${calibration['sensor_kit_base_link']['traffic_light_left_camera/camera_link']['y']}"
-      z="${calibration['sensor_kit_base_link']['traffic_light_left_camera/camera_link']['z']}"
-      roll="${calibration['sensor_kit_base_link']['traffic_light_left_camera/camera_link']['roll']}"
-      pitch="${calibration['sensor_kit_base_link']['traffic_light_left_camera/camera_link']['pitch']}"
-      yaw="${calibration['sensor_kit_base_link']['traffic_light_left_camera/camera_link']['yaw']}"
-      fps="30"
-      width="800"
-      height="400"
-      fov="1.3"
-    />
-    <xacro:monocular_camera_macro
-      name="camera0/camera"
-      parent="sensor_kit_base_link"
-      namespace=""
-      x="${calibration['sensor_kit_base_link']['camera0/camera_link']['x']}"
-      y="${calibration['sensor_kit_base_link']['camera0/camera_link']['y']}"
-      z="${calibration['sensor_kit_base_link']['camera0/camera_link']['z']}"
-      roll="${calibration['sensor_kit_base_link']['camera0/camera_link']['roll']}"
-      pitch="${calibration['sensor_kit_base_link']['camera0/camera_link']['pitch']}"
-      yaw="${calibration['sensor_kit_base_link']['camera0/camera_link']['yaw']}"
-      fps="30"
-      width="800"
-      height="400"
-      fov="1.3"
-    />
-    <xacro:monocular_camera_macro
-      name="camera1/camera"
-      parent="sensor_kit_base_link"
-      namespace=""
-      x="${calibration['sensor_kit_base_link']['camera1/camera_link']['x']}"
-      y="${calibration['sensor_kit_base_link']['camera1/camera_link']['y']}"
-      z="${calibration['sensor_kit_base_link']['camera1/camera_link']['z']}"
-      roll="${calibration['sensor_kit_base_link']['camera1/camera_link']['roll']}"
-      pitch="${calibration['sensor_kit_base_link']['camera1/camera_link']['pitch']}"
-      yaw="${calibration['sensor_kit_base_link']['camera1/camera_link']['yaw']}"
-      fps="30"
-      width="800"
-      height="400"
-      fov="1.3"
-    />
-    <xacro:monocular_camera_macro
-      name="camera2/camera"
-      parent="sensor_kit_base_link"
-      namespace=""
-      x="${calibration['sensor_kit_base_link']['camera2/camera_link']['x']}"
-      y="${calibration['sensor_kit_base_link']['camera2/camera_link']['y']}"
-      z="${calibration['sensor_kit_base_link']['camera2/camera_link']['z']}"
-      roll="${calibration['sensor_kit_base_link']['camera2/camera_link']['roll']}"
-      pitch="${calibration['sensor_kit_base_link']['camera2/camera_link']['pitch']}"
-      yaw="${calibration['sensor_kit_base_link']['camera2/camera_link']['yaw']}"
-      fps="30"
-      width="800"
-      height="400"
-      fov="1.3"
-    />
-    <xacro:monocular_camera_macro
-      name="camera3/camera"
-      parent="sensor_kit_base_link"
-      namespace=""
-      x="${calibration['sensor_kit_base_link']['camera3/camera_link']['x']}"
-      y="${calibration['sensor_kit_base_link']['camera3/camera_link']['y']}"
-      z="${calibration['sensor_kit_base_link']['camera3/camera_link']['z']}"
-      roll="${calibration['sensor_kit_base_link']['camera3/camera_link']['roll']}"
-      pitch="${calibration['sensor_kit_base_link']['camera3/camera_link']['pitch']}"
-      yaw="${calibration['sensor_kit_base_link']['camera3/camera_link']['yaw']}"
-      fps="30"
-      width="800"
-      height="400"
-      fov="1.3"
-    />
-    <xacro:monocular_camera_macro
-      name="camera4/camera"
-      parent="sensor_kit_base_link"
-      namespace=""
-      x="${calibration['sensor_kit_base_link']['camera4/camera_link']['x']}"
-      y="${calibration['sensor_kit_base_link']['camera4/camera_link']['y']}"
-      z="${calibration['sensor_kit_base_link']['camera4/camera_link']['z']}"
-      roll="${calibration['sensor_kit_base_link']['camera4/camera_link']['roll']}"
-      pitch="${calibration['sensor_kit_base_link']['camera4/camera_link']['pitch']}"
-      yaw="${calibration['sensor_kit_base_link']['camera4/camera_link']['yaw']}"
-      fps="30"
-      width="800"
-      height="400"
-      fov="1.3"
-    />
-    <xacro:monocular_camera_macro
-      name="camera5/camera"
-      parent="sensor_kit_base_link"
-      namespace=""
-      x="${calibration['sensor_kit_base_link']['camera5/camera_link']['x']}"
-      y="${calibration['sensor_kit_base_link']['camera5/camera_link']['y']}"
-      z="${calibration['sensor_kit_base_link']['camera5/camera_link']['z']}"
-      roll="${calibration['sensor_kit_base_link']['camera5/camera_link']['roll']}"
-      pitch="${calibration['sensor_kit_base_link']['camera5/camera_link']['pitch']}"
-      yaw="${calibration['sensor_kit_base_link']['camera5/camera_link']['yaw']}"
-      fps="30"
-      width="800"
-      height="400"
-      fov="1.3"
-    /> -->
-    <!-- gnss -->
-    <xacro:imu_macro
-      name="gnss"
-      parent="sensor_kit_base_link"
-      namespace=""
-      x="${calibration['sensor_kit_base_link']['gnss_link']['x']}"
-      y="${calibration['sensor_kit_base_link']['gnss_link']['y']}"
-      z="${calibration['sensor_kit_base_link']['gnss_link']['z']}"
-      roll="${calibration['sensor_kit_base_link']['gnss_link']['roll']}"
-      pitch="${calibration['sensor_kit_base_link']['gnss_link']['pitch']}"
-      yaw="${calibration['sensor_kit_base_link']['gnss_link']['yaw']}"
-      fps="100"
-    />
-    <!-- imu -->
-    <xacro:imu_macro
-      name="tamagawa/imu"
-      parent="sensor_kit_base_link"
-      namespace=""
-      x="${calibration['sensor_kit_base_link']['tamagawa/imu_link']['x']}"
-      y="${calibration['sensor_kit_base_link']['tamagawa/imu_link']['y']}"
-      z="${calibration['sensor_kit_base_link']['tamagawa/imu_link']['z']}"
-      roll="${calibration['sensor_kit_base_link']['tamagawa/imu_link']['roll']}"
-      pitch="${calibration['sensor_kit_base_link']['tamagawa/imu_link']['pitch']}"
-      yaw="${calibration['sensor_kit_base_link']['tamagawa/imu_link']['yaw']}"
-      fps="100"
-    />
+             ${calibration['sensor_kit_base_link']['velodyne_right_base_link']['yaw']}"/>
+    </joint>
+    <link name="velodyne_left"/>
+    <joint name="velodyne_left_joint" type="fixed">
+      <parent link="velodyne_left_base_link"/>
+      <child link="velodyne_left"/>
+      <origin xyz="0 0 0" rpy="0 0 0"/>
+    </joint>
+    <link name="velodyne_right"/>
+    <joint name="velodyne_right_joint" type="fixed">
+      <parent link="velodyne_right_base_link"/>
+      <child link="velodyne_right"/>
+      <origin xyz="0 0 0" rpy="0 0 0"/>
+    </joint>
+    <!-- Primary IMU left Livox's internal IMU, kept under the legacy frame id
+         `tamagawa/imu_link` so imu_corrector / EKF / rviz configs don't change.
+         Datasheet offset (MID-360 LiDAR optical centre -> internal IMU, in the
+         LiDAR's native non-inverted frame) x=-0.011, y=-0.02329, z=0.04412.
+         The LiDAR's roll=π inversion is inherited by this IMU child.
+         The Livox driver must publish IMU messages with frame_id = tamagawa/imu_link
+         (or be remapped before imu_corrector) for the TF lookup to match. -->
+    <link name="tamagawa/imu_link"/>
+    <joint name="tamagawa_imu_link_joint" type="fixed">
+      <parent link="velodyne_left_base_link"/>
+      <child link="tamagawa/imu_link"/>
+      <origin xyz="-0.011 -0.02329 0.04412" rpy="0 0 0"/>
+    </joint>
   </xacro:macro>
 </robot>

File: sensor_kit/autoware_towtruck_sensor_kit_launch/autoware_towtruck_sensor_kit_description/urdf/sensors.xacro (robot description, xacro)
@@ -15,6 +15,6 @@
   />
   <!-- embedded sensors -->
-  <!-- <xacro:include filename="$(find velodyne_description)/urdf/VLP-16.urdf.xacro"/>
-  <xacro:VLP-16 parent="base_link" name="velodyne_rear" topic="velodyne_rear/velodyne_points" hz="10" samples="220" gpu="false">
+  <!-- <xacro include filename="$(find velodyne_description)/urdf/VLP-16.urdf.xacro"/>
+  <xacroVLP-16 parent="base_link" name="velodyne_rear" topic="velodyne_rear/velodyne_points" hz="10" samples="220" gpu="false">
     <origin
       xyz="${calibration['base_link']['velodyne_rear_base_link']['x']}
@@ -25,4 +25,4 @@
            ${calibration['base_link']['velodyne_rear_base_link']['yaw']}"
     />
-  </xacro:VLP-16> -->
+  </xacroVLP-16> -->
 </robot>

File: vehicle/autoware_towtruck_vehicle_launch/autoware_towtruck_vehicle_description/urdf/vehicle.xacro (robot description, xacro)
@@ -2,19 +2,26 @@
 <robot xmlns:xacro="http://ros.org/wiki/xacro" name="basic_mobile_bot">
   <xacro:property name="vehicle_info" value="${xacro.load_yaml('$(find autoware_towtruck_vehicle_description)/config/vehicle_info.param.yaml')}"/>
-  <xacro:property name="base_width" value="0.78"/>
-  <xacro:property name="base_length" value="1.27"/>
-  <xacro:property name="base_height" value="1.90"/>
-  <xacro:property name="wheel_radius" value="0.2"/>
-  <xacro:property name="wheel_width" value="0.09"/>
-  <xacro:property name="wheel_ygap" value="0.01"/>
-  <xacro:property name="wheel_zoff" value="0.05"/>
-  <xacro:property name="wheel_xoff" value="0.635"/>
-  <xacro:property name="steering_wheel_xoff" value="0.55"/>
+  <!-- geometric constants (m) -->
+  <xacro:property name="body_length" value="1.52"/>
+  <xacro:property name="body_width" value="0.79"/>
+  <xacro:property name="body_height" value="1.83"/>
+  <xacro:property name="body_x_centre" value="0.435"/>   <!-- (-rear_overhang + body_length/2) = -0.325 + 0.76 -->
+  <xacro:property name="body_z_centre" value="0.915"/>   <!-- body box spans z = 0 .. 1.83 (absorbs 0.07 ground clearance) -->
+  <xacro:property name="rear_wheel_radius" value="0.195"/>
+  <xacro:property name="rear_wheel_width" value="0.095"/>
+  <xacro:property name="rear_wheel_y" value="0.3475"/>   <!-- wheel_tread/2 = 0.695/2 -->
+  <xacro:property name="front_wheel_radius" value="0.12"/>
+  <xacro:property name="front_wheel_width" value="0.24"/>
+  <xacro:property name="front_wheel_x" value="0.995"/>   <!-- wheel_base -->
+  <xacro:property name="max_steer" value="0.9774"/>
+  <!-- mirror geometry & placement -->
+  <xacro:property name="mirror_x" value="0.12"/>
+  <xacro:property name="mirror_y" value="0.01"/>
+  <xacro:property name="mirror_z" value="0.20"/>
+  <xacro:property name="mirror_centre_x" value="1.067"/>
+  <xacro:property name="mirror_centre_y" value="0.635"/>
+  <xacro:property name="mirror_centre_z" value="1.51"/>
   <link name="base_link"/>
-  <joint name="chassis_joint" type="fixed">
-    <parent link="base_link"/>
-    <child link="chassis_link"/>
-    <origin xyz="${wheel_xoff} 0 ${wheel_zoff}" rpy="0 0 0"/>
-  </joint>
+  <!-- chassis (body box) -->
   <link name="chassis_link">
     <inertial>
@@ -24,7 +31,7 @@
     </inertial>
     <visual>
-      <origin xyz="0 0 0.95" rpy="0 0 0"/>
+      <origin xyz="0 0 0" rpy="0 0 0"/>
       <geometry>
-        <box size="${base_length} ${base_width} ${base_height}"/>
+        <box size="${body_length} ${body_width} ${body_height}"/>
       </geometry>
       <material name="Red">
@@ -32,11 +39,23 @@
       </material>
     </visual>
+    <collision>
+      <origin xyz="0 0 0" rpy="0 0 0"/>
+      <geometry>
+        <box size="${body_length} ${body_width} ${body_height}"/>
+      </geometry>
+    </collision>
   </link>
-  <xacro:macro name="wheel" params="prefix y_reflect">
+  <joint name="chassis_joint" type="fixed">
+    <parent link="base_link"/>
+    <child link="chassis_link"/>
+    <origin xyz="${body_x_centre} 0 ${body_z_centre}" rpy="0 0 0"/>
+  </joint>
+  <!-- rear wheels (drive, no steering) -->
+  <xacro:macro name="rear_wheel" params="prefix y_reflect">
     <link name="${prefix}_link">
       <visual>
         <origin xyz="0 0 0" rpy="${pi/2} 0 0"/>
         <geometry>
-            <cylinder radius="${wheel_radius}" length="${wheel_width}"/>
+          <cylinder radius="${rear_wheel_radius}" length="${rear_wheel_width}"/>
         </geometry>
         <material name="White">
@@ -48,15 +67,16 @@
       <parent link="base_link"/>
       <child link="${prefix}_link"/>
-      <origin xyz="0 ${y_reflect*(base_width/2+wheel_ygap)} 0" rpy="0 0 0"/>
+      <origin xyz="0 ${y_reflect * rear_wheel_y} ${rear_wheel_radius}" rpy="0 0 0"/>
       <axis xyz="0 1 0"/>
     </joint>
   </xacro:macro>
-  <xacro:wheel prefix="drivewhl_l" y_reflect="1" />
-  <xacro:wheel prefix="drivewhl_r" y_reflect="-1" />
+  <xacro:rear_wheel prefix="drivewhl_l" y_reflect="1"/>
+  <xacro:rear_wheel prefix="drivewhl_r" y_reflect="-1"/>
+  <!-- front single (dual-modelled) steering wheel -->
   <link name="steering_link"/>
   <joint name="steering_joint" type="fixed">
-    <parent link="chassis_link"/>
+    <parent link="base_link"/>
     <child link="steering_link"/>
-    <origin xyz="${steering_wheel_xoff} 0 -${wheel_zoff}" rpy="0 0 0"/>
+    <origin xyz="${front_wheel_x} 0 ${front_wheel_radius}" rpy="0 0 0"/>
   </joint>
   <link name="front_steering_wheel_link">
@@ -64,5 +84,5 @@
       <origin xyz="0 0 0" rpy="${pi/2} 0 0"/>
       <geometry>
-        <cylinder radius="${wheel_radius}" length="${wheel_width}"/>
+        <cylinder radius="${front_wheel_radius}" length="${front_wheel_width}"/>
       </geometry>
       <material name="White">
@@ -75,6 +95,34 @@
     <child link="front_steering_wheel_link"/>
     <origin xyz="0 0 0" rpy="0 0 0"/>
-    <limit upper="1.047" lower="-1.047" effort="10" velocity="1.0"/>
+    <limit upper="${max_steer}" lower="${-max_steer}" effort="10" velocity="1.0"/>
     <axis xyz="0 0 1"/>
   </joint>
+  <!-- mirrors -->
+  <xacro:macro name="mirror_panel" params="prefix y_reflect">
+    <link name="${prefix}_link">
+      <visual>
+        <origin xyz="0 0 0" rpy="0 0 0"/>
+        <geometry>
+          <box size="${mirror_x} ${mirror_y} ${mirror_z}"/>
+        </geometry>
+        <material name="Grey">
+          <color rgba="0.4 0.4 0.4 1.0"/>
+        </material>
+      </visual>
+      <collision>
+        <origin xyz="0 0 0" rpy="0 0 0"/>
+        <geometry>
+          <box size="${mirror_x} ${mirror_y} ${mirror_z}"/>
+        </geometry>
+      </collision>
+    </link>
+    <joint name="${prefix}_joint" type="fixed">
+      <parent link="base_link"/>
+      <child link="${prefix}_link"/>
+      <!-- TODO verify mirror X — assumes mirror face aligns with sloped body front at mirror mid-height -->
+      <origin xyz="${mirror_centre_x} ${y_reflect * mirror_centre_y} ${mirror_centre_z}" rpy="0 0 0"/>
+    </joint>
+  </xacro:macro>
+  <xacro:mirror_panel prefix="mirror_left" y_reflect="1"/>
+  <xacro:mirror_panel prefix="mirror_right" y_reflect="-1"/>
 </robot>
